Commit message: added some world examples

File: urdf/robotic_hand.xacro (robot description, xacro)
@@ -6,4 +6,5 @@
   <xacro:property name="pi" value="3.1415926" />
   <xacro:property name="max_speed" value="0.5" />
+  <xacro:property name="max_effort" value="10000000" />
   <!-- Used for fixing robot to Gazebo 'base_link' -->
   <link name="world"/>
@@ -104,5 +105,5 @@
       lower="-3.1416"
       upper="3.1416"
-      effort="10000000"
+      effort="${max_effort}"
       velocity="${max_speed}" />
   </joint>
@@ -169,5 +170,5 @@
       lower="-3.1416"
       upper="0.57"
-      effort="1000000"
+      effort="${max_effort}"
       velocity="${max_speed}" />
   </joint>
@@ -234,5 +235,5 @@
       lower="-0.55"
       upper="1.50"
-      effort="10000000"
+      effort="${max_effort}"
       velocity="${max_speed}" />
   </joint>
@@ -299,5 +300,5 @@
       lower="-0.50"
       upper="1.57"
-      effort="99999"
+      effort="${max_effort}"
       velocity="${max_speed}" />
   </joint>
